File: eagle/midi_to_cv.brd (EAGLE design)
At the start: 100 x 80 mm, 21 parts, among them IC1 4067N, U1 ATMEGA328P_PDIP

Commit message: panel for resonant eq controller
Parts:
- removed JP2: M16LONGPADS, SparkFun-Connectors:1X16_LONGPADS
- added D2: (no value), SparkFun-DiscreteSemi:DIODE-1N4148
- added JP1: (no value), SparkFun-Connectors:2X3-NS
- added JP3, JP4, JP5, JP6: (no value), SparkFun-Connectors:1X04_LONGPADS
- added OK1: 6N138, optocoupler:DIL08
- added PAD1: midi pin 4, wirepad:2,54/0,9
- added PAD2: midi pin 5, wirepad:2,54/0,9
- added R2, R5: 220, rcl:0207/10
- added R3: 270, rcl:0207/10
- added R7: 1M, rcl:0207/10
- moved IC1 62.3 mm to (83.6, 32.0), turned to 180 degrees
- moved C3 61.7 mm to (68.3, 18.5), turned to 270 degrees
- moved MIDI4 58.0 mm to (19.3, 18.3)
- moved C2 56.4 mm to (59.4, 24.4), turned to 90 degrees
- moved MIDI2 52.9 mm to (41.4, 15.7)
- moved Q1 49.4 mm to (51.1, 24.6), turned to 180 degrees
- moved MIDI5 46.7 mm to (21.1, 27.4)
- moved R1 41.3 mm to (33.3, 23.9), turned to 180 degrees
- moved C1 40.5 mm to (42.9, 24.1), turned to 90 degrees
- moved RESET1 37.8 mm to (25.1, 23.9)
- moved R6 36.8 mm to (28.7, 27.2), turned to 180 degrees
- moved U1 24.0 mm to (41.9, 34.8), turned to 0 degrees
- moved RESET2 23.9 mm to (25.4, 43.9)
- moved U$1 20.0 mm to (56.9, 6.86), turned to 0 degrees
- moved POT_5V 18.0 mm to (62.5, 14.7)
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Connections:
- new net N$29: D2.A, OK1.3, PAD2.1
- new net N$30: D2.C, OK1.2, R2.2
- new net N$31: PAD1.1, R2.1
- new net N$32: OK1.6, R3.1, U1.2
- new net N$33: MIDI4.1, R5.2
- new net N$34: JP1.4, U1.17
- new net N$36: JP1.1, U1.18
- net +5V: now also JP1.2, OK1.8, R3.2, R5.1; no longer MIDI5.1
- net GND: now also JP1.6, OK1.5
- net N$1: now also JP1.5
- net N$10: now also JP1.3
- net N$12: now also U1.12; no longer U1.16
- net N$13: now also U1.13; no longer U1.17
- net N$14: now also U1.14; no longer U1.18
- net N$15: now also JP5.4; no longer JP2.5
- net N$17: now also JP5.3; no longer JP2.6
- net N$19: now also JP5.2; no longer JP2.7
- net N$2: now also JP6.4; no longer JP2.1
- net N$20: now also JP5.1; no longer JP2.8
- net N$21: now also JP4.4; no longer JP2.9
- net N$22: now also JP4.3; no longer JP2.10
- net N$23: now also JP4.2; no longer JP2.11
- net N$24: now also JP4.1; no longer JP2.12
- net N$25: now also JP3.4; no longer JP2.13
- net N$26: now also JP3.3; no longer JP2.14
- net N$27: now also JP3.2; no longer JP2.15
- net N$28: now also JP3.1; no longer JP2.16
- net N$3: now also JP6.3; no longer JP2.2
- net N$4: now also R7.2
- net N$5: now also R7.1
- net N$6: now also MIDI5.1; no longer MIDI4.1
- net N$7: now also JP6.2; no longer JP2.3
- net N$8: now also JP6.1; no longer JP2.4
- net N$9: now also U1.11; no longer U1.15
Routing:
- net N$1: track 15.1 -> 66.0 mm, vias 0 -> 2
- net N$14: track 60.4 -> 20.2 mm
- net N$10: track 7.49 -> 41.5 mm
- net GND: track 276.6 -> 246.5 mm, vias 2 -> 0
- net N$2: track 34.3 -> 6.09 mm
- net N$28: track 34.0 -> 5.90 mm
- net N$3: track 31.0 -> 5.72 mm
- net N$27: track 31.1 -> 5.91 mm
- net N$36: track 0.00 -> 22.9 mm
- net N$7: track 27.8 -> 5.70 mm
- net N$26: track 28.0 -> 5.96 mm
- net N$25: track 25.5 -> 5.93 mm
- net N$8: track 25.3 -> 5.82 mm
- net N$32: track 0.00 -> 18.9 mm
- net N$15: track 23.0 -> 5.74 mm
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Other:
- outline, holes or cut-outs redrawn

Commit message: code working in hardware
Parts:
- renumbered MIDI2 to MOUT_P2, MIDI4 to MOUT_P4, MIDI5 to MOUT_P5, PAD1 to MIN_P4, PAD2 to MIN_P5
Changed lines of the file:
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@@
 <element name="RESET2" library="wirepad" package="2,54/0,9" value="reset " x="25.4" y="43.942"/>
 <element name="LED_NEG" library="wirepad" package="2,54/0,9" value="gate LED" x="34.036" y="43.688"/>
-<element name="MIDI5" library="wirepad" package="2,54/0,9" value="midi out pin 5" x="21.082" y="27.432"/>
-<element name="MIDI4" library="wirepad" package="2,54/0,9" value="midi out pin 4" x="19.304" y="18.288"/>
-<element name="MIDI2" library="wirepad" package="2,54/0,9" value="midi out pin 2" x="41.402" y="15.748"/>
+<element name="MOUT_P5" library="wirepad" package="2,54/0,9" value="midi out pin 5" x="21.082" y="27.432"/>
+<element name="MOUT_P4" library="wirepad" package="2,54/0,9" value="midi out pin 4" x="19.304" y="18.288"/>
+<element name="MOUT_P2" library="wirepad" package="2,54/0,9" value="midi out pin 2" x="41.402" y="15.748"/>
 <element name="Q1" library="crystal" package="HC49U-V" value="" x="51.054" y="24.638" rot="R180">
 <attribute name="OC_NEWARK" value="unknown" x="51.054" y="24.638" size="1.778" layer="27" rot="R180" display="off"/>
@@
 </element>
 <element name="R2" library="rcl" package="0207/10" value="220" x="25.4" y="9.652" rot="R270"/>
-<element name="PAD1" library="wirepad" package="2,54/0,9" value="midi pin 4" x="21.336" y="4.318"/>
-<element name="PAD2" library="wirepad" package="2,54/0,9" value="midi pin 5" x="40.64" y="4.318"/>
+<element name="MIN_P4" library="wirepad" package="2,54/0,9" value="midi pin 4" x="21.336" y="4.318"/>
+<element name="MIN_P5" library="wirepad" package="2,54/0,9" value="midi pin 5" x="40.64" y="4.318"/>
 <element name="R3" library="rcl" package="0207/10" value="270" x="29.972" y="20.32" rot="R180"/>
 <element name="R5" library="rcl" package="0207/10" value="220" x="22.352" y="12.446" rot="R90"/>
@@
 <contactref element="IC1" pad="12"/>
 <contactref element="C4" pad="2"/>
-<contactref element="MIDI2" pad="1"/>
+<contactref element="MOUT_P2" pad="1"/>
 <contactref element="IC1" pad="15"/>
 <contactref element="POT_GRN" pad="1"/>
@@
 <signal name="N$6">
 <contactref element="R6" pad="2"/>
-<contactref element="MIDI5" pad="1"/>
+<contactref element="MOUT_P5" pad="1"/>
 <wire x1="21.082" y1="27.432" x2="23.5712" y2="27.432" width="0.5588" layer="16"/>
 <wire x1="23.5712" y1="27.432" x2="23.622" y2="27.178" width="0.5588" layer="16"/>
@@
 <signal name="N$29">
 <contactref element="OK1" pad="3"/>
-<contactref element="PAD2" pad="1"/>
+<contactref element="MIN_P5" pad="1"/>
 <contactref element="D2" pad="A"/>
 <wire x1="35.306" y1="3.429" x2="35.306" y2="7.1628" width="0.5588" layer="16"/>
@@
 </signal>
 <signal name="N$31">
-<contactref element="PAD1" pad="1"/>
+<contactref element="MIN_P4" pad="1"/>
 <contactref element="R2" pad="1"/>
 <wire x1="25.1714" y1="6.6294" x2="25.1714" y2="14.6304" width="0.5588" layer="16"/>
@@
 <signal name="N$33">
 <contactref element="R5" pad="2"/>
-<contactref element="MIDI4" pad="1"/>
+<contactref element="MOUT_P4" pad="1"/>
 <wire x1="19.304" y1="17.8308" x2="21.971" y2="17.8308" width="0.5588" layer="16"/>
 <wire x1="21.971" y1="17.8308" x2="22.352" y2="17.526" width="0.5588" layer="16"/>
