File: eagle/midi_to_cv.sch (EAGLE design)
At the start: 21 parts, among them IC1 4067N, U1 ATMEGA328P_PDIP

Commit message: panel for resonant eq controller
Parts:
- removed JP2: M16LONGPADS, SparkFun-Connectors:M16LONGPADS
- added D2: (no value), SparkFun-DiscreteSemi:DIODE1N4148
- added JP1: (no value), SparkFun-Connectors:M03X2NO_SILK
- added JP3, JP4, JP5, JP6: (no value), SparkFun-Connectors:M04LONGPADS
- added OK1: 6N138, optocoupler:6N138
- added PAD1: midi pin 4, wirepad:2,54/0,9
- added PAD2: midi pin 5, wirepad:2,54/0,9
- added R2, R5: 220, rcl:R-US_0207/10
- added R3: 270, rcl:R-US_0207/10
- added R7: 1M, rcl:R-US_0207/10
Connections:
- new net N$29: D2.A, OK1.C, PAD2.P
- new net N$30: D2.C, OK1.A, R2.2
- new net N$31: PAD1.P, R2.1
- new net N$32: OK1.VO, R3.1, U1.PD0(RXD)
- new net N$33: MIDI4.P, R5.2
- new net N$34: JP1.4, U1.PB3(MOSI/OC2)
- new net N$36: JP1.1, U1.PB4(MISO)
- net +5V: now also JP1.2, OK1.VCC, R3.2, R5.1; no longer MIDI5.P
- net GND: now also JP1.6, OK1.GND
- net N$1: now also JP1.5
- net N$10: now also JP1.3
- net N$12: now also U1.PD6(AIN0); no longer U1.PB2(SS/OC1B)
- net N$13: now also U1.PD7(AIN1); no longer U1.PB3(MOSI/OC2)
- net N$14: now also U1.PB0(ICP); no longer U1.PB4(MISO)
- net N$15: now also JP5.4; no longer JP2.5
- net N$17: now also JP5.3; no longer JP2.6
- net N$19: now also JP5.2; no longer JP2.7
- net N$2: now also JP6.4; no longer JP2.1
- net N$20: now also JP5.1; no longer JP2.8
- net N$21: now also JP4.4; no longer JP2.9
- net N$22: now also JP4.3; no longer JP2.10
- net N$23: now also JP4.2; no longer JP2.11
- net N$24: now also JP4.1; no longer JP2.12
- net N$25: now also JP3.4; no longer JP2.13
- net N$26: now also JP3.3; no longer JP2.14
- net N$27: now also JP3.2; no longer JP2.15
- net N$28: now also JP3.1; no longer JP2.16
- net N$3: now also JP6.3; no longer JP2.2
- net N$4: now also R7.2
- net N$5: now also R7.1
- net N$6: now also MIDI5.P; no longer MIDI4.P
- net N$7: now also JP6.2; no longer JP2.3
- net N$8: now also JP6.1; no longer JP2.4
- net N$9: now also U1.PD5(T1); no longer U1.PB1(OC1A)
Other:
- moved on the sheet: C4, IC1P, MIDI2, MIDI4, MIDI5, POT_5V, POT_GRN, R6, U$1

Commit message: code working in hardware
Parts:
- renumbered MIDI2 to MOUT_P2, MIDI4 to MOUT_P4, MIDI5 to MOUT_P5, PAD1 to MIN_P4, PAD2 to MIN_P5
Changed lines of the file:
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@@
 <part name="GND4" library="supply1" deviceset="GND" device=""/>
 <part name="R6" library="rcl" deviceset="R-US_" device="0207/10" value="220"/>
-<part name="MIDI5" library="wirepad" deviceset="2,54/0,9" device="" value="midi out pin 5"/>
-<part name="MIDI4" library="wirepad" deviceset="2,54/0,9" device="" value="midi out pin 4"/>
-<part name="MIDI2" library="wirepad" deviceset="2,54/0,9" device="" value="midi out pin 2"/>
+<part name="MOUT_P5" library="wirepad" deviceset="2,54/0,9" device="" value="midi out pin 5"/>
+<part name="MOUT_P4" library="wirepad" deviceset="2,54/0,9" device="" value="midi out pin 4"/>
+<part name="MOUT_P2" library="wirepad" deviceset="2,54/0,9" device="" value="midi out pin 2"/>
 <part name="GND2" library="supply1" deviceset="GND" device=""/>
 <part name="P+2" library="supply1" deviceset="+5V" device=""/>
@@
 <part name="OK1" library="optocoupler" deviceset="6N138" device=""/>
 <part name="R2" library="rcl" deviceset="R-US_" device="0207/10" value="220"/>
-<part name="PAD1" library="wirepad" deviceset="2,54/0,9" device="" value="midi pin 4"/>
-<part name="PAD2" library="wirepad" deviceset="2,54/0,9" device="" value="midi pin 5"/>
+<part name="MIN_P4" library="wirepad" deviceset="2,54/0,9" device="" value="midi pin 4"/>
+<part name="MIN_P5" library="wirepad" deviceset="2,54/0,9" device="" value="midi pin 5"/>
 <part name="R3" library="rcl" deviceset="R-US_" device="0207/10" value="270"/>
 <part name="P+7" library="supply1" deviceset="+5V" device=""/>
@@
 <instance part="GND4" gate="1" x="43.18" y="104.14"/>
 <instance part="R6" gate="G$1" x="58.42" y="116.84"/>
-<instance part="MIDI5" gate="1" x="78.74" y="116.84" rot="R180"/>
-<instance part="MIDI4" gate="1" x="78.74" y="132.08" rot="R180"/>
-<instance part="MIDI2" gate="1" x="71.12" y="124.46" rot="R180"/>
+<instance part="MOUT_P5" gate="1" x="78.74" y="116.84" rot="R180"/>
+<instance part="MOUT_P4" gate="1" x="78.74" y="132.08" rot="R180"/>
+<instance part="MOUT_P2" gate="1" x="71.12" y="124.46" rot="R180"/>
 <instance part="GND2" gate="1" x="81.28" y="35.56"/>
 <instance part="P+2" gate="1" x="93.98" y="132.08"/>
@@
 <instance part="OK1" gate="G$1" x="-12.7" y="121.92"/>
 <instance part="R2" gate="G$1" x="-43.18" y="127"/>
-<instance part="PAD1" gate="1" x="-58.42" y="127"/>
-<instance part="PAD2" gate="1" x="-58.42" y="116.84"/>
+<instance part="MIN_P4" gate="1" x="-58.42" y="127"/>
+<instance part="MIN_P5" gate="1" x="-58.42" y="116.84"/>
 <instance part="R3" gate="G$1" x="15.24" y="127" rot="R90"/>
 <instance part="P+7" gate="1" x="5.08" y="142.24"/>
@@
 <wire x1="30.48" y1="109.22" x2="43.18" y2="109.22" width="0.1524" layer="91"/>
 <junction x="43.18" y="109.22"/>
-<pinref part="MIDI2" gate="1" pin="P"/>
+<pinref part="MOUT_P2" gate="1" pin="P"/>
 <wire x1="68.58" y1="124.46" x2="48.26" y2="124.46" width="0.1524" layer="91"/>
 <wire x1="48.26" y1="124.46" x2="48.26" y2="109.22" width="0.1524" layer="91"/>
@@
 <segment>
 <pinref part="R6" gate="G$1" pin="2"/>
-<pinref part="MIDI5" gate="1" pin="P"/>
+<pinref part="MOUT_P5" gate="1" pin="P"/>
 <wire x1="76.2" y1="116.84" x2="63.5" y2="116.84" width="0.1524" layer="91"/>
 </segment>
@@
 <wire x1="-25.4" y1="116.84" x2="-33.02" y2="116.84" width="0.1524" layer="91"/>
 <wire x1="-33.02" y1="116.84" x2="-33.02" y2="119.38" width="0.1524" layer="91"/>
-<pinref part="PAD2" gate="1" pin="P"/>
+<pinref part="MIN_P5" gate="1" pin="P"/>
 <wire x1="-55.88" y1="116.84" x2="-33.02" y2="116.84" width="0.1524" layer="91"/>
 <junction x="-33.02" y="116.84"/>
@@
 <net name="N$31" class="0">
 <segment>
-<pinref part="PAD1" gate="1" pin="P"/>
+<pinref part="MIN_P4" gate="1" pin="P"/>
 <pinref part="R2" gate="G$1" pin="1"/>
 <wire x1="-55.88" y1="127" x2="-48.26" y2="127" width="0.1524" layer="91"/>
@@
 <segment>
 <pinref part="R5" gate="G$1" pin="2"/>
-<pinref part="MIDI4" gate="1" pin="P"/>
+<pinref part="MOUT_P4" gate="1" pin="P"/>
 <wire x1="60.96" y1="132.08" x2="76.2" y2="132.08" width="0.1524" layer="91"/>
 </segment>
